Commit message: fix: validate all Gazebo simulation scenarios

File: simulation/ros2_ws/src/r680_sim_description/urdf/r680_sim.urdf.xacro (robot description, xacro)
@@ -2,5 +2,4 @@
 <robot xmlns:xacro="http://www.ros.org/wiki/xacro" name="r680_sim">
   <!-- Simulation assumptions only. Replace after physical R680 measurement. -->
-  <xacro:property name="pi" value="3.141592653589793"/>
   <xacro:property name="wheel_radius" value="0.10"/>
   <xacro:property name="wheel_width" value="0.05"/>
@@ -78,5 +77,5 @@
   </gazebo>
   <gazebo reference="c16_link">
-    <sensor name="c16_sim" type="gpu_ray"><always_on>true</always_on><update_rate>10</update_rate><visualize>false</visualize>
+    <sensor name="c16_sim" type="ray"><always_on>true</always_on><update_rate>10</update_rate><visualize>false</visualize>
       <ray><scan>
         <horizontal><samples>900</samples><resolution>1</resolution><min_angle>-${pi}</min_angle><max_angle>${pi}</max_angle></horizontal>

Commit message: feat: add stage3 C16 feature bridge and control configs

File: simulation/ros2_ws/src/r680_sim_description/urdf/r680_sim.urdf.xacro (robot description, xacro)
@@ -1,4 +1,5 @@
 <?xml version="1.0"?>
 <robot xmlns:xacro="http://www.ros.org/wiki/xacro" name="r680_sim">
+  <xacro:arg name="use_ros2_control" default="false"/>
   <!-- Simulation assumptions only. Replace after physical R680 measurement. -->
   <xacro:property name="wheel_radius" value="0.10"/>
@@ -59,5 +60,5 @@
   <gazebo reference="front_caster_link"><mu1>0.05</mu1><mu2>0.05</mu2></gazebo>
   <gazebo reference="rear_caster_link"><mu1>0.05</mu1><mu2>0.05</mu2></gazebo>
-  <gazebo>
+  <gazebo if="$(eval arg('use_ros2_control') == 'false')">
     <plugin name="r680_diff_drive" filename="libgazebo_ros_diff_drive.so">
       <ros><namespace>/</namespace><remapping>cmd_vel:=cmd_vel</remapping><remapping>odom:=odom</remapping></ros>
@@ -67,4 +68,21 @@
       <publish_odom>true</publish_odom><publish_odom_tf>true</publish_odom_tf><publish_wheel_tf>true</publish_wheel_tf>
       <odometry_frame>odom</odometry_frame><robot_base_frame>base_footprint</robot_base_frame>
+    </plugin>
+  </gazebo>
+  <ros2_control name="GazeboSystem" type="system" if="$(eval arg('use_ros2_control') == 'true')">
+    <hardware><plugin>gazebo_ros2_control/GazeboSystem</plugin></hardware>
+    <joint name="left_wheel_joint">
+      <command_interface name="velocity"><param name="min">-12.0</param><param name="max">12.0</param></command_interface>
+      <state_interface name="position"/><state_interface name="velocity"/>
+    </joint>
+    <joint name="right_wheel_joint">
+      <command_interface name="velocity"><param name="min">-12.0</param><param name="max">12.0</param></command_interface>
+      <state_interface name="position"/><state_interface name="velocity"/>
+    </joint>
+  </ros2_control>
+  <gazebo if="$(eval arg('use_ros2_control') == 'true')">
+    <plugin name="gazebo_ros2_control" filename="libgazebo_ros2_control.so">
+      <robot_param>robot_description</robot_param><robot_param_node>robot_state_publisher</robot_param_node>
+      <parameters>$(find r680_sim_description)/config/controllers.yaml</parameters>
     </plugin>
   </gazebo>

Commit message: Complete Nav2 ros2_control simulation loop

File: simulation/ros2_ws/src/r680_sim_description/urdf/r680_sim.urdf.xacro (robot description, xacro)
@@ -60,31 +60,35 @@
   <gazebo reference="front_caster_link"><mu1>0.05</mu1><mu2>0.05</mu2></gazebo>
   <gazebo reference="rear_caster_link"><mu1>0.05</mu1><mu2>0.05</mu2></gazebo>
-  <gazebo unless="$(arg use_ros2_control)">
-    <plugin name="r680_diff_drive" filename="libgazebo_ros_diff_drive.so">
-      <ros><namespace>/</namespace><remapping>cmd_vel:=cmd_vel</remapping><remapping>odom:=odom</remapping></ros>
-      <update_rate>50</update_rate><left_joint>left_wheel_joint</left_joint><right_joint>right_wheel_joint</right_joint>
-      <wheel_separation>${wheel_separation}</wheel_separation><wheel_diameter>${2 * wheel_radius}</wheel_diameter>
-      <max_wheel_torque>45</max_wheel_torque><max_wheel_acceleration>1.0</max_wheel_acceleration>
-      <publish_odom>true</publish_odom><publish_odom_tf>true</publish_odom_tf><publish_wheel_tf>true</publish_wheel_tf>
-      <odometry_frame>odom</odometry_frame><robot_base_frame>base_footprint</robot_base_frame>
-    </plugin>
-  </gazebo>
-  <ros2_control name="GazeboSystem" type="system" if="$(arg use_ros2_control)">
-    <hardware><plugin>gazebo_ros2_control/GazeboSystem</plugin></hardware>
-    <joint name="left_wheel_joint">
-      <command_interface name="velocity"><param name="min">-12.0</param><param name="max">12.0</param></command_interface>
-      <state_interface name="position"/><state_interface name="velocity"/>
-    </joint>
-    <joint name="right_wheel_joint">
-      <command_interface name="velocity"><param name="min">-12.0</param><param name="max">12.0</param></command_interface>
-      <state_interface name="position"/><state_interface name="velocity"/>
-    </joint>
-  </ros2_control>
-  <gazebo if="$(arg use_ros2_control)">
-    <plugin name="gazebo_ros2_control" filename="libgazebo_ros2_control.so">
-      <robot_param>robot_description</robot_param><robot_param_node>robot_state_publisher</robot_param_node>
-      <parameters>$(find r680_sim_description)/config/controllers.yaml</parameters>
-    </plugin>
-  </gazebo>
+  <xacro:unless value="$(arg use_ros2_control)">
+    <gazebo>
+      <plugin name="r680_diff_drive" filename="libgazebo_ros_diff_drive.so">
+        <ros><namespace>/</namespace><remapping>cmd_vel:=cmd_vel</remapping><remapping>odom:=odom</remapping></ros>
+        <update_rate>50</update_rate><left_joint>left_wheel_joint</left_joint><right_joint>right_wheel_joint</right_joint>
+        <wheel_separation>${wheel_separation}</wheel_separation><wheel_diameter>${2 * wheel_radius}</wheel_diameter>
+        <max_wheel_torque>45</max_wheel_torque><max_wheel_acceleration>1.0</max_wheel_acceleration>
+        <publish_odom>true</publish_odom><publish_odom_tf>true</publish_odom_tf><publish_wheel_tf>true</publish_wheel_tf>
+        <odometry_frame>odom</odometry_frame><robot_base_frame>base_footprint</robot_base_frame>
+      </plugin>
+    </gazebo>
+  </xacro:unless>
+  <xacro:if value="$(arg use_ros2_control)">
+    <ros2_control name="GazeboSystem" type="system">
+      <hardware><plugin>gazebo_ros2_control/GazeboSystem</plugin></hardware>
+      <joint name="left_wheel_joint">
+        <command_interface name="velocity"><param name="min">-12.0</param><param name="max">12.0</param></command_interface>
+        <state_interface name="position"/><state_interface name="velocity"/>
+      </joint>
+      <joint name="right_wheel_joint">
+        <command_interface name="velocity"><param name="min">-12.0</param><param name="max">12.0</param></command_interface>
+        <state_interface name="position"/><state_interface name="velocity"/>
+      </joint>
+    </ros2_control>
+    <gazebo>
+      <plugin name="gazebo_ros2_control" filename="libgazebo_ros2_control.so">
+        <robot_param>robot_description</robot_param><robot_param_node>robot_state_publisher</robot_param_node>
+        <parameters>$(find r680_sim_description)/config/controllers.yaml</parameters>
+      </plugin>
+    </gazebo>
+  </xacro:if>
   <gazebo reference="laser_2d_link">
     <sensor name="safety_scan" type="ray"><always_on>true</always_on><update_rate>15</update_rate><visualize>false</visualize>
